File: hardware/project/ETH1CJTAG/ETH1CJTAG.kicad_pcb (KiCad board)
At the start: 4 copper layers, 160 x 100 mm, 451 parts, among them J1101 Conn_01x02, J1102 Conn_01x03_Male, J301 693071010811, J401 105133-0001, J601 Conn_02x05, J801 C64AC, K601 TQ2SA-5V, K602 TQ2SA-5V, K701 TQ2SA-5V, K702 TQ2SA-5V, K703 TQ2SA-5V, K704 TQ2SA-5V, K705 TQ2SA-5V, Q501 IRFR5410, Q502 TSM2323, Q601 MMBT3904, Q602 MMBT3904, Q603 BC847, Q701 2SD1048, Q702 BC847, Q703 BC847, Q704 BC847, Q705 BC847, SW1101 TDA06H0B1, U1001 TLC272, U1002 TLC272, U1003 ADS7828, U1004 TLC272, U1005 TLC272, U1101 chiliSOM, U201 LC03-3.3, U202 LAN8720A, U203 LC03-3.3, U204 82400274, U301 82400274, U302 82400274, U401 824011, U402 824011, U403 FT230XQ, U404 824011, U501 TPS61073, U502 TPS61073, U503 TEL 10-2411WI, U504 MAX5902, U505 TEL 10-2415WI, U506 AQY212GS, U601 LT3080EQ, U602 LM334M, U603 TLC272, U604 AQY212GS, U605 MAX4080FASA+, U606 MCP3204, U607 TLC272, U608 TLC272, U609 MCP4922-ESL, U610 REF3025, U611 AP1117-33, U612 STM32F405RGT6, U613 24LC256, U701 NC7SZ125, U702 NC7SZ125, U703 NC7SZ125, U704 FT2232H, U705 93LC56, U706 NC7SZ125, U707 AP1117E33G-13, U708 NC7SZ125, U709 NC7SZ125, U710 AQY212GS, U711 NC7SZ125, U712 IRF7455, U713 NC7SZ125, U901 74AC125, U902 SN74LVC1T45DBV, U903 ADuM5402, U904 SN74LVC1T45DBV, U905 SN74LVC1T45DBV, U906 AQY212GS, Y201 ECS-250-8-36CKM-TR, Y601 ECS-120-8-36-CKM-TR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

Commit message: PCB design
Parts:
- added C1105: 100n, ETH1CJTAG:C_0603_A_Pad1.05x0.95mm_HandSolder, F.Cu at (235.7, 13.2)
- added J1103: Conn_02x10_Counter_Clockwise, Connector_PinHeader_1.27mm:PinHeader_2x10_P1.27mm_Vertical_SMD, F.Cu at (88.9, 102.7)
- added R1145: 0, ETH1CJTAG:R_0603_E_Pad1.05x0.95mm_HandSolder, F.Cu at (240.1, 13.2)
- added R1147: 49R9, Resistor_SMD:R_0603_1608Metric_Pad1.05x0.95mm_HandSolder, F.Cu at (235.7, 15.7)
- added R1148: 10k, ETH1CJTAG:R_0603_G_Pad1.05x0.95mm_HandSolder, F.Cu at (235.7, 18.2)
- added R701: 22, ETH1CJTAG:R_0603_H_Pad1.05x0.95mm_HandSolder, F.Cu at (135.1, 85.4)
- added R733: 22, ETH1CJTAG:R_0603_H_Pad1.05x0.95mm_HandSolder, F.Cu at (136.7, 85.4)
- C201, C202, C207, C208, C209, C210, C211, C215, C502, C506, R1105, R1106, R1110, R1111, R1112, R1113, R1114, R1115, R1117, R1118, R1119, R1120, R1121, R1122, R1123, R1124, R1125, R1128, R1129, R1130, R1131, R1132, R1133, R1134, R1135, R1136, R1137, R1138, R1139, R1140, R1141, R1142, R1143, R201, R202, R203, R204, R213, R214, R217, R218, R219, R301, R302, R303, R304, R305, R306, R501, R502, R504, R506, R508, R509, R713, Y601, Y701: moved to B.Cu
- U701, U702, U703, U706, U708, U709, U711, U713: footprint Package_TO_SOT_SMD:SOT-353_SC-70-5_Handsoldering -> Package_TO_SOT_SMD:SOT-353_SC-70-5
- moved L501 433.5 mm to (100.2, 87.4)
- moved R501 432.3 mm to (105.0, 85.9)
- moved R502 421.6 mm to (105.0, 88.6), turned to 180 degrees
- moved R301 414.8 mm to (82.8, 86.7)
- moved U501 411.7 mm to (105.0, 87.4), turned to 90 degrees
- moved R305 411.1 mm to (82.8, 77.7)
- moved R506 410.1 mm to (128.5, 89.0), turned to 180 degrees
- moved R303 409.4 mm to (82.8, 83.7)
- moved R304 405.6 mm to (82.8, 79.2)
- moved R302 405.3 mm to (82.8, 85.2)
- moved R306 404.8 mm to (82.8, 88.3)
- moved L502 404.0 mm to (123.6, 87.6)
- moved R504 403.9 mm to (128.5, 86.0)
- moved U502 399.3 mm to (128.5, 87.6), turned to 90 degrees
- moved C502 396.5 mm to (108.5, 87.4), turned to 270 degrees
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Connections:
- C711 pad 1: USB0_VCC -> USB1_VCC
- L401 pad 1: /SOM/USB1_D_N -> /SOM/USB1_D_P
- L401 pad 2: /JTAG/F_USB1_D_N -> /JTAG/F_USB1_D_P
- L401 pad 3: /JTAG/F_USB1_D_P -> /JTAG/F_USB1_D_N
- L401 pad 4: /SOM/USB1_D_P -> /SOM/USB1_D_N
- U1101 pad 157: (no net) -> /SOM/chili_~TRST
- U1101 pad 158: (no net) -> /SOM/chili_TCK
- U1101 pad 159: (no net) -> /SOM/chili_TDO
- U1101 pad 160: (no net) -> /SOM/chili_TDI
- U1101 pad 161: (no net) -> /SOM/chili_TMS
- U1101 pad 8: (no net) -> /SOM/chili_RESETn
- U704 pad 7: /JTAG/F_USB1_D_P -> Net-(R701-Pad1)
- U704 pad 8: /JTAG/F_USB1_D_N -> Net-(R733-Pad1)
- U707 pad 3: USB0_VCC -> USB1_VCC
- Y601 pad 1: Net-(C624-Pad1) -> Net-(C625-Pad1)
- Y601 pad 3: Net-(C625-Pad1) -> Net-(C624-Pad1)

Commit message: PCB layout
Parts:
- removed the C1004 at (381.5, 123.4)
- removed the C710 at (466.1, 49.7)
- removed the C714 at (462.0, 47.2)
- removed the C716 at (469.2, 41.5)
- removed the C720 at (484.9, 27.5)
- removed the D707 at (448.8, 44.8)
- removed the R702 at (152.9, 59.1)
- removed the R723 at (470.6, 33.9)
- removed the U707 at (142.1, 60.3)
- removed the U708 at (168.2, 22.5)
- removed the U712 at (151.1, 27.9)
- added C709: 8p, ETH1CJTAG:C_0603_S_Pad1.05x0.95mm_HandSolder, B.Cu at (134.5, 80.8)
- added C712: 100n, ETH1CJTAG:C_0603_A_Pad1.05x0.95mm_HandSolder, F.Cu at (143.0, 58.0)
- added C715: 100n, ETH1CJTAG:C_0603_A_Pad1.05x0.95mm_HandSolder, F.Cu at (157.7, 58.0)
- added C719: 100n, ETH1CJTAG:C_0603_A_Pad1.05x0.95mm_HandSolder, B.Cu at (165.4, 68.8)
- added D714: BAT54S, Package_TO_SOT_SMD:SOT-23, F.Cu at (166.0, 64.4)
- added R701: 82, ETH1CJTAG:R_0603_F_Pad1.05x0.95mm_HandSolder, F.Cu at (161.4, 58.0)
- added R724: 22k, Resistor_SMD:R_0603_1608Metric_Pad1.05x0.95mm_HandSolder, F.Cu at (150.2, 58.0)
- added U705: NC7SZ125, Package_TO_SOT_SMD:SOT-353_SC-70-5, F.Cu at (165.4, 68.7)
- added U711: TLV75533PDBV, Package_TO_SOT_SMD:SOT-23-5, F.Cu at (127.0, 66.7)
- added U713: IRF7455, Package_SO:SO-8_3.9x4.9mm_P1.27mm, F.Cu at (136.8, 60.7)
- C1001, C1102, C1103, C1104, C1105, C206, C212, C213, C214, C301, C302, C303, C304, C401, C410, C411, C412, C413, C414, C501, C504, C505, C507, C512, C513, C518, C603, C604, C605, C606, C608, C609, C611, C612, C616, C617, C618, C619, C620, C621, C624, C625, C626, C627, C628, C629, C630, C631, C632, C701, C702, C713, D601, D604, FB601, FB701, FID102, FID104, J1103, Q601, Q602, Q603, Q701, Q702, Q703, Q704, R1001, R1002, R1003, R1004, R1005, R1006, R1007, R1008, R1009, R1010, R1011, R1012, R1013, R1014, R1015, R1016, R1101, R1102, R1103, R1104, R1107, R1108, R1116, R1126, R1127, R1144, R1145, R1146, R1147, R1148, R503, R505, R602, R604, R605, R606, R607, R608, R609, R610, R611, R612, R613, R614, R615, R616, R617, R618, R619, R620, R621, R622, R623, R624, R625, R628, R629, R630, R631, R632, R633, Y201, Y602: moved to B.Cu
- C1004: renamed from C1005; moved to B.Cu
- C1005: renamed from C1006; moved to B.Cu
- C1006: renamed from C1007; moved to B.Cu
- C1007: renamed from C1008; moved to B.Cu
- C1008: renamed from C1009; moved to B.Cu
- C1009: renamed from C1010; moved to B.Cu
- C506: moved to F.Cu
- C703: renamed from C704; moved to B.Cu
- C704: renamed from C705; moved to B.Cu
- C705: renamed from C706; moved to B.Cu
- C706: renamed from C707; moved to B.Cu
- C708: renamed from C709; moved to B.Cu
- C720: renamed from C721; moved to B.Cu
- C721: renamed from C722; moved to B.Cu
- C722: renamed from C723; moved to B.Cu
- C723: renamed from C724; moved to B.Cu
- C724: renamed from C725; moved to B.Cu
- C725: renamed from C726; moved to B.Cu
- D1102: footprint Diode_SMD:D_SOD-323_HandSoldering -> Diode_SMD:D_SOD-323; moved to B.Cu
- D502, D505, D603, D901: footprint Diode_SMD:D_SMB_Handsoldering -> Diode_SMD:D_SMB
- D709: renamed from D710; moved to B.Cu
- D710: renamed from D711; moved to B.Cu
- D711: renamed from D712; moved to B.Cu
- D712: renamed from D713; moved to B.Cu
- D713: renamed from D714; moved to B.Cu
- L1101: value SDE1006A-180M -> 851-CDRH74NP-180MC; footprint ETH1CJTAG:SDE1006A -> ETH1CJTAG:CDRH74
- R705: renamed from R706; moved to B.Cu
- R707: renamed from R708; moved to B.Cu
- R715: renamed from R714; moved to B.Cu
- R716: renamed from R715; moved to B.Cu
- R719: renamed from R718; moved to B.Cu
- R720: renamed from R719; moved to B.Cu
- R721: renamed from R720; moved to B.Cu
- R722: renamed from R721; moved to B.Cu
- R723: renamed from R722; moved to B.Cu
- R727: renamed from R726; moved to B.Cu
- R728: renamed from R727; moved to B.Cu
- R729: renamed from R728; moved to B.Cu
- R730: renamed from R729; moved to B.Cu
- R732: renamed from R731; moved to B.Cu
- R733: renamed from R732; moved to B.Cu
- U204, U301, U302: footprint Package_TO_SOT_SMD:SOT-363_SC-70-6_Handsoldering -> Package_TO_SOT_SMD:SOT-363_SC-70-6
- U401, U402, U404: footprint Package_TO_SOT_SMD:SOT-23-5_HandSoldering -> Package_TO_SOT_SMD:SOT-23-5
- U501, U502: footprint Package_TO_SOT_SMD:SOT-23-6_Handsoldering -> Package_TO_SOT_SMD:SOT-23-6
- U611: value AP1117-33 -> TLV75533PDBV; footprint Package_TO_SOT_SMD:SOT-223-3_TabPin2 -> Package_TO_SOT_SMD:SOT-23-5
- moved C501 428.9 mm to (108.5, 88.8), turned to 270 degrees
- moved R503 410.2 mm to (105.0, 91.6), turned to 180 degrees
- moved C304 410.1 mm to (77.6, 97.0), turned to 180 degrees
- moved C303 407.1 mm to (84.6, 97.9)
- moved C302 401.1 mm to (94.6, 101.0)
- moved U302 399.0 mm to (94.6, 101.0), turned to 90 degrees
- moved C301 397.0 mm to (94.6, 96.5)
- moved R511 393.4 mm to (149.7, 132.1), turned to 180 degrees
- moved U301 393.2 mm to (94.6, 96.5), turned to 270 degrees
- moved C504 391.6 mm to (128.5, 84.8)
- moved R505 388.2 mm to (131.8, 89.0), turned to 270 degrees
- moved R512 384.0 mm to (149.7, 130.3), turned to 180 degrees
- moved C505 379.8 mm to (125.1, 88.8), turned to 270 degrees
- moved C629 360.6 mm to (102.6, 64.3), turned to 180 degrees
- moved C615 357.1 mm to (96.0, 71.9)
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- renumbered C708 to C707, C711 to C710, C712 to C711, C715 to C714, C717 to C716, C718 to C717, C719 to C718, D704 to D701, D705 to D702, D706 to D703, D703 to D704, D701 to D705, D702 to D706, D708 to D707, D709 to D708, R703 to R702, R704 to R703, R705 to R704, R707 to R706, R709 to R708, R710 to R709, R711 to R710, R701 to R711, R733 to R712, R712 to R713, R713 to R714, R716 to R717, R717 to R718, R724 to R725, R725 to R726, R730 to R731, U706 to U704, U704 to U706, U709 to U707, U705 to U708, U711 to U709, U713 to U710, U710 to U712
Connections:
- net /Connector/TSRST renamed /Connector/SRST
- net /JTAG/TSRST1 renamed /JTAG/SRST1
- net /JTAG/TSRST1_A renamed /JTAG/SRST1_A
- D709 pad 2: /JTAG/JTAG_REL3 -> /JTAG/JTAG_REL2
- D710 pad 2: /JTAG/JTAG_REL1 -> /JTAG/JTAG_REL2
- D712 pad 2: /JTAG/JTAG_REL2 -> /JTAG/JTAG_REL1
- D713 pad 2: /JTAG/JTAG_REL2 -> /JTAG/JTAG_REL3
- K701 pad 10: /JTAG/JTAG_REL3 -> /JTAG/JTAG_REL2
- K702 pad 10: /JTAG/JTAG_REL1 -> /JTAG/JTAG_REL2
- K704 pad 10: /JTAG/JTAG_REL2 -> /JTAG/JTAG_REL1
- K705 pad 10: /JTAG/JTAG_REL2 -> /JTAG/JTAG_REL3
- U611 pad 1: GNDA -> USB0_VCC
- U611 pad 2: Net-(C614-Pad1) -> GNDA

Commit message: PCB layout
Parts:
- added J802: 615008145221, ETH1CJTAG:615008145221, F.Cu at (199.8, 96.0)
- C413, C414, C704, Q701, R707, R715: moved to F.Cu
- C622, C623, R212, R220, R221, R222: moved to B.Cu
- moved C212 35.7 mm to (124.7, 97.5), turned to 90 degrees
- moved D712 30.7 mm to (213.5, 63.4)
- moved K704 30.6 mm to (208.4, 63.4)
- moved K705 30.5 mm to (177.9, 63.4)
- moved D713 30.5 mm to (183.0, 63.5)
- moved R715 26.8 mm to (165.3, 72.3), turned to 0 degrees
- moved R716 21.9 mm to (157.7, 65.3), turned to 0 degrees
- moved Q703 15.3 mm to (176.9, 63.4)
- moved R729 15.3 mm to (174.1, 63.4)
- moved Q704 15.1 mm to (191.9, 63.4)
- moved R732 15.1 mm to (189.1, 63.4)
- moved C409 14.6 mm to (150.1, 108.2), turned to 270 degrees
- moved R220 11.5 mm to (152.7, 92.1), turned to 0 degrees
- moved C214 10.6 mm to (162.3, 91.8), turned to 90 degrees
- moved C705 9.94 mm to (129.5, 73.4), turned to 270 degrees
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Connections:
- J801 pad A20: /Connector/RX- -> /Connector/RX+
- J801 pad A21: /Connector/RX+ -> /Connector/RX-
- J801 pad C20: /Connector/TX- -> /Connector/TX+
- J801 pad C21: /Connector/TX+ -> /Connector/TX-
- U612 pad 16: (no net) -> /PSU/CLIM
- U612 pad 26: /PSU/CLIM -> (no net)
Routing:
- net /JTAG/TMS1: track 0.00 -> 64.3 mm, vias 0 -> 2
- net /Connector/SRST: track 0.00 -> 63.2 mm
- net /JTAG/TDI1: track 0.00 -> 57.5 mm, vias 0 -> 2
- net /JTAG/nRESET1: track 0.00 -> 55.2 mm, vias 0 -> 3
- net /Connector/nRESET: track 0.00 -> 55.1 mm
- net /JTAG/TCK1: track 0.00 -> 53.1 mm, vias 0 -> 2
- net /JTAG/TDO1: track 0.00 -> 50.9 mm, vias 0 -> 2
- net /SOM/DBG_RXD: track 0.00 -> 49.9 mm, vias 0 -> 1
- net /SOM/DBG_TXD: track 0.00 -> 49.7 mm, vias 0 -> 1
- net /Connector/TRST: track 0.00 -> 49.3 mm
- net USB0_VBUS: track 0.00 -> 47.0 mm, vias 0 -> 1
- net Net-(C602-Pad1): track 0.00 -> 46.3 mm
- net /SOM/SD_CD: track 0.00 -> 45.9 mm, vias 0 -> 1
- net /Connector/RCTK: track 0.00 -> 45.7 mm
- net /JTAG/RCTK1: track 0.00 -> 43.7 mm
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- added copper zone on GND, net GNDPWR
Other:
- net class Default: clearance 0.2 -> 0.127; trace_width 0.25 -> 0.127; via_dia 0.8 -> 0.5; via_drill 0.4 -> 0.2
- rule trace_clearance: 0.2 -> 0.127
- rule trace_min: 0.2 -> 0.127
- rule via_min_drill: 0.3 -> 0.15
- rule via_min_size: 0.4 -> 0.5
- board text added: "1"
- board text added: "2"
- board text added: "3"
- board text added: "4"
- board text added: "ETH1CJTAG PROTOTYP V1.0 IP: 192.168.1.123 PORT: 2000"

Commit message: PCB layout
Parts:
- U204: moved to B.Cu
- moved C206 11.3 mm to (165.0, 102.4)
- moved U204 4.32 mm to (169.7, 96.1), turned to 0 degrees
- moved R212 3.28 mm to (160.3, 94.9), turned to 0 degrees
- moved C205 2.80 mm to (160.4, 102.6)
- moved C203 2.58 mm to (165.0, 104.3)
- moved FB201 2.55 mm to (160.4, 104.3)
- moved C204 2.34 mm to (165.0, 102.4)
- moved C210 1.87 mm to (169.8, 99.2), turned to 0 degrees
- moved R203 1.87 mm to (169.8, 97.9), turned to 0 degrees
- moved R204 1.87 mm to (169.8, 100.5), turned to 0 degrees
- moved R201 1.78 mm to (169.7, 91.6)
- moved C207 1.78 mm to (169.7, 92.8), turned to 0 degrees
- moved R202 1.78 mm to (169.7, 94.1), turned to 0 degrees
- moved U201 1.02 mm to (184.7, 93.2)
- moved U203 1.02 mm to (184.7, 98.8)
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Routing:
- net /Connector/TX+: track 0.00 -> 41.4 mm
- net /Connector/TX-: track 0.00 -> 40.6 mm
- net /Connector/RX+: track 0.00 -> 37.5 mm
- net /Connector/RX-: track 0.00 -> 33.3 mm
- net (no net): track 30.5 -> 0.00 mm
- net /Ethernet/ETH_RD_N: track 0.00 -> 20.3 mm, vias 0 -> 3
- net /Ethernet/ETH_TD_P: track 0.00 -> 19.1 mm, vias 0 -> 1
- net /Ethernet/ETH_RD_P: track 0.00 -> 18.9 mm, vias 0 -> 3
- net Net-(C203-Pad1): track 33.4 -> 16.0 mm
- net /Ethernet/ETH_TD_N: track 0.00 -> 14.5 mm, vias 0 -> 1
- net Net-(L201-Pad14): track 0.00 -> 4.00 mm
- net Net-(L201-Pad11): track 0.00 -> 3.98 mm
- net Net-(L201-Pad9): track 0.00 -> 3.68 mm
- net Net-(L201-Pad16): track 0.00 -> 3.67 mm
- net Net-(R212-Pad2): track 1.40 -> 0.00 mm, vias 1 -> 0
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- added copper zone on Power, net GNDPWR
- removed copper zone on GND, net GNDPWR

Commit message: PCB layout
Parts:
- C503, C506: moved to B.Cu
- C505: moved to F.Cu
- moved D1101 60.6 mm to (144.3, 131.0), turned to 180 degrees
- moved R1105 60.0 mm to (144.9, 130.0), turned to 180 degrees
- moved R1107 59.5 mm to (141.4, 132.1), turned to 180 degrees
- moved R1106 57.0 mm to (141.4, 130.0), turned to 180 degrees
- moved C503 31.6 mm to (100.2, 88.8)
- moved C506 8.26 mm to (123.6, 88.9), turned to 270 degrees
- moved C505 6.74 mm to (131.8, 89.1)
- moved FB602 1.89 mm to (90.4, 72.8), turned to 0 degrees
- moved D711 0.63 mm to (198.2, 63.4)
- moved D1102 0.46 mm to (91.7, 120.5)
- moved L1101 0.46 mm to (91.7, 120.5)
- moved C1102 0.46 mm to (95.0, 120.5)
- moved C406 0.38 mm to (117.5, 90.6)
- moved C721 0.26 mm to (132.9, 75.7)
- moved L502 0.25 mm to (123.6, 88.8)
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Connections:
- U1101 pad 101: (no net) -> /JTAG/JTAG_REL_CTR2
- U1101 pad 131: /SOM/LED_GREEN -> (no net)
- U1101 pad 132: /SOM/LED_RED -> (no net)
- U1101 pad 133: /SOM/LED_BLUE -> (no net)
- U1101 pad 136: Net-(C1101-Pad1) -> (no net)
- U1101 pad 145: /Power/ENA_24V_PSU -> (no net)
- U1101 pad 148: /JTAG/JTAG_REL_CTR1 -> (no net)
- U1101 pad 149: /JTAG/JTAG_REL_CTR3 -> (no net)
- U1101 pad 155: /JTAG/JTAG_REL_CTR2 -> Net-(C1101-Pad1)
- U1101 pad 46: (no net) -> /Power/ENA_24V_PSU
- U1101 pad 47: (no net) -> /SOM/LED_BLUE
- U1101 pad 48: (no net) -> /SOM/LED_RED
- U1101 pad 49: (no net) -> /SOM/LED_GREEN
- U1101 pad 96: (no net) -> /JTAG/JTAG_REL_CTR1
- U1101 pad 98: (no net) -> /JTAG/JTAG_REL_CTR3
Routing:
- net /JTAG/JTAG_REL_CTR2: track 0.00 -> 100.8 mm, vias 0 -> 1
- net /JTAG/JTAG_REL_CTR1: track 0.00 -> 87.2 mm, vias 0 -> 1
- net /SOM/TRIG_EN: track 0.00 -> 85.4 mm, vias 0 -> 4
- net /SOM/TRIG_OUT: track 0.00 -> 83.5 mm, vias 0 -> 4
- net /JTAG/3V3_JTAG_CTR: track 0.00 -> 79.9 mm, vias 0 -> 7
- net /SOM/TRIG_IN: track 0.00 -> 76.9 mm, vias 0 -> 4
- net +3.3V_JTAG: track 0.00 -> 73.3 mm, vias 0 -> 36
- net /JTAG/JTAG_REL_CTR3: track 0.00 -> 72.6 mm, vias 0 -> 1
- net Net-(R621-Pad2): track 0.00 -> 69.4 mm, vias 0 -> 3
- net /JTAG/nRESET_OUT: track 0.00 -> 67.4 mm, vias 0 -> 3
- net /SOM/ENA_5V_TRIG: track 0.00 -> 65.9 mm, vias 0 -> 4
- net /JTAG/FT_~RESET: track 0.00 -> 64.8 mm, vias 0 -> 4
- net +3.3V_D: track 6.35 -> 60.2 mm, vias 0 -> 17
- net /PSU/PSU_SENSE: track 0.00 -> 52.8 mm, vias 0 -> 2
- net GNDA: track 3.47 -> 54.2 mm, vias 2 -> 39
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- added copper zone on Power, net 5V_TRIG
- added copper zone on B.Cu, net GND
- added copper zone on F.Cu, net GND
- added copper zone on GND, net GND
- added copper zone on B.Cu, net GNDA
- added copper zone on F.Cu, net GNDA
- added copper zone on GND, net GNDA
- added copper zone on GND, net GNDS

Commit message: PCB layout
Parts:
- moved R1105 55.2 mm to (89.7, 129.7), turned to 0 degrees
- moved D1101 54.2 mm to (90.2, 128.7), turned to 0 degrees
- moved R1107 48.4 mm to (93.2, 127.6), turned to 0 degrees
- moved R1106 48.2 mm to (93.2, 129.7), turned to 0 degrees
- moved SW1101 13.8 mm to (81.4, 120.7)
- moved C516 8.52 mm to (154.8, 134.0), turned to 180 degrees
- moved R1118 6.47 mm to (119.9, 124.6)
- moved R1120 6.47 mm to (114.8, 124.6)
- moved R1133 6.47 mm to (119.9, 121.2)
- moved R1136 6.47 mm to (114.8, 121.2)
- moved R1117 6.47 mm to (126.2, 121.2)
- moved R1119 6.47 mm to (116.1, 121.2)
- moved R1121 6.47 mm to (113.5, 124.6)
- moved R1122 6.47 mm to (112.3, 124.6)
- moved R1123 6.47 mm to (111.0, 124.6)
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Routing:
- net /Connector/SENSE: track 0.00 -> 66.6 mm, vias 0 -> 2
- net +24V_PSU: track 11.4 -> 58.8 mm, vias 1 -> 19
- net +2V5: track 10.3 -> 49.4 mm
- net GNDA: track 54.2 -> 87.8 mm, vias 39 -> 59
- net Net-(C602-Pad1): track 46.3 -> 75.3 mm, vias 0 -> 17
- net +1.8V_JTAG: track 10.5 -> 35.2 mm
- net +3.3V_JTAG: track 73.3 -> 95.9 mm, vias 36 -> 39
- net +5VD: track 22.2 -> 44.5 mm, vias 8 -> 21
- net +3.3V_PSU: track 36.4 -> 56.9 mm, vias 14 -> 18
- net Net-(R1124-Pad1): track 11.6 -> 30.0 mm
- net Net-(C513-Pad2): track 0.00 -> 18.1 mm, vias 0 -> 4
- net Net-(R1122-Pad1): track 13.5 -> 31.6 mm
- net Net-(R1123-Pad1): track 12.6 -> 30.7 mm
- net Net-(R1125-Pad1): track 10.8 -> 28.8 mm
- net Net-(R1121-Pad1): track 15.0 -> 32.6 mm
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- added copper zone on Power, net +1.8V_JTAG
- added copper zone on B.Cu, net +24V_PSU
- added copper zone on F.Cu, net +24V_PSU
- added copper zone on Power, net +24V_PSU
- added copper zone on Power, net +3.3V_D
- added copper zone on Power, net +3.3V_JTAG
- added copper zone on Power, net +3.3V_PSU
- added copper zone on Power, net +3.3V_TEST
- added copper zone on B.Cu, net +5VD
- added copper zone on F.Cu, net +5VD
- added copper zone on Power, net +5VD
- added copper zone on B.Cu, net /Connector/+VOUT
- added copper zone on F.Cu, net /Connector/+VOUT
- added copper zone on Power, net /Connector/+VOUT
- added copper zone on B.Cu, net /Connector/-VOUT
- added copper zone on F.Cu, net /Connector/-VOUT
- added copper zone on GND, net /Connector/-VOUT
- added copper zone on Power, net 3.3V_DBG
- added copper zone on Power, net 5V_ISO_TRIG
- added copper zone on B.Cu, net 5V_USB
- added copper zone on F.Cu, net 5V_USB
- added copper zone on Power, net 5V_USB
- added copper zone on Power, net DBG_USB_VCC
- added copper zone on B.Cu, net Net-(C513-Pad2)
- added copper zone on F.Cu, net Net-(C513-Pad2)
- added copper zone on B.Cu, net Net-(C515-Pad1)
- added copper zone on F.Cu, net Net-(C515-Pad1)
- added copper zone on B.Cu, net Net-(C516-Pad1)
- added copper zone on F.Cu, net Net-(C516-Pad1)
- added copper zone on Power, net Net-(C516-Pad1)
- added copper zone on B.Cu, net Net-(C602-Pad1)
- added copper zone on F.Cu, net Net-(C602-Pad1)
- added copper zone on Power, net Net-(C602-Pad1)
- added copper zone on B.Cu, net Net-(C603-Pad1)
- added copper zone on F.Cu, net Net-(C603-Pad1)
- added copper zone on Power, net Net-(C603-Pad1)
- removed copper zone on Power, net 5V_TRIG
