File: hardware/project/ETH1CJTAG/ETH1CJTAG.kicad_pcb (KiCad board)
At the start: 4 copper layers, 160 x 100 mm, 458 parts, among them J1101 Conn_01x02, J1102 Conn_01x03_Male, J1103 Conn_02x10_Counter_Clockwise, J301 693071010811, J401 105133-0001, J601 Conn_02x05, J801 C64AC, J802 615008145221, K601 TQ2SA-5V, K602 TQ2SA-5V, K701 TQ2SA-5V, K702 TQ2SA-5V, K703 TQ2SA-5V, K704 TQ2SA-5V, K705 TQ2SA-5V, Q501 IRFR5410, Q502 TSM2323, Q601 MMBT3904, Q602 MMBT3904, Q603 BC847, Q701 2SD1048, Q702 BC847, Q703 BC847, Q704 BC847, Q705 BC847, SW1101 TDA06H0B1, U1001 TLC272, U1002 TLC272, U1003 ADS7828, U1004 TLC272, U1005 TLC272, U1101 chiliSOM, U201 LC03-3.3, U202 LAN8720A, U203 LC03-3.3, U204 82400274, U301 82400274, U302 82400274, U401 824011, U402 824011, U403 FT230XQ, U404 824011, U501 TPS61073, U502 TPS61073, U503 TEL 10-2411WI, U504 MAX5902, U505 TEL 10-2415WI, U506 AQY212GS, U601 LT3080EQ, U602 LM334M, U603 TLC272, U604 AQY212GS, U605 MAX4080FASA+, U606 MCP3204, U607 TLC272, U608 TLC272, U609 MCP4922-ESL, U610 REF3025, U611 TLV75533PDBV, U612 STM32F405RGT6, U613 24LC256, U701 NC7SZ125, U702 NC7SZ125, U703 NC7SZ125, U704 NC7SZ125, U705 NC7SZ125, U706 FT2232H, U707 NC7SZ125, U708 93LC56, U709 NC7SZ125, U710 NC7SZ125, U711 TLV75533PDBV, U712 AQY212GS, U713 IRF7455, U901 74AC125, U902 SN74LVC1T45DBV, U903 ADuM5402, U904 SN74LVC1T45DBV, U905 SN74LVC1T45DBV, U906 AQY212GS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

Commit message: PCB layout
Parts:
- moved R1128 3.68 mm to (131.2, 121.2)
- moved R1117 3.43 mm to (129.7, 121.2)
- moved R1129 3.17 mm to (128.1, 121.2)
- moved R1130 2.92 mm to (126.6, 121.2)
- moved D503 2.70 mm to (211.6, 125.0)
- moved R1131 2.67 mm to (125.1, 121.2)
- moved R1132 2.41 mm to (123.6, 121.2)
- moved R1118 2.16 mm to (122.0, 124.6)
- moved R1133 2.16 mm to (122.0, 121.2)
- moved R1134 1.91 mm to (120.5, 121.2)
- moved R1135 1.65 mm to (119.0, 121.2)
- moved R208 1.40 mm to (152.7, 90.7)
- moved R220 1.40 mm to (152.7, 90.7)
- moved R1119 1.40 mm to (117.5, 121.2)
- moved R908 1.35 mm to (150.0, 87.0)
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Connections:
- U1101 pad 28: (no net) -> /SOM/LED_BLUE
- U1101 pad 29: (no net) -> /SOM/LED_RED
- U1101 pad 30: (no net) -> /SOM/LED_GREEN
- U1101 pad 47: /SOM/LED_BLUE -> (no net)
- U1101 pad 48: /SOM/LED_RED -> (no net)
- U1101 pad 49: /SOM/LED_GREEN -> (no net)
Routing:
- net GNDA: track 87.8 -> 203.6 mm, vias 59 -> 94
- net +3.3V_D: track 74.2 -> 163.6 mm, vias 21 -> 31
- net +3.3VA: track 0.00 -> 63.4 mm, vias 0 -> 2
- net Net-(K701-Pad3): track 0.30 -> 63.6 mm, vias 0 -> 4
- net /Connector/-VOUT: track 16.8 -> 72.3 mm
- net Net-(C508-Pad1): track 0.00 -> 44.7 mm, vias 0 -> 14
- net /SOM/LED_RED: track 0.00 -> 35.7 mm, vias 0 -> 1
- net /SOM/LED_BLUE: track 0.00 -> 33.5 mm, vias 0 -> 1
- net /SOM/LED_GREEN: track 0.00 -> 32.7 mm, vias 0 -> 1
- net /SOM/SD_CD: track 45.9 -> 18.2 mm, vias 1 -> 0
- net GNDPWR: track 0.00 -> 16.8 mm, vias 0 -> 2
- net Net-(D503-Pad1): track 0.00 -> 13.6 mm, vias 0 -> 8
- net 5V_USB: track 6.78 -> 18.7 mm, vias 3 -> 12
- net Net-(D504-Pad2): track 0.00 -> 8.75 mm, vias 0 -> 1
- net Net-(J1103-Pad5): track 8.73 -> 0.00 mm
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- added copper zone on B.Cu, net +24V
- added copper zone on F.Cu, net +24V
- added copper zone on Power, net +24V
- added copper zone on F.Cu, net +3.3V_D
- added copper zone on GND, net GNDPWR
- added copper zone on B.Cu, net Net-(C507-Pad1)
- added copper zone on F.Cu, net Net-(C507-Pad1)
- added copper zone on Power, net Net-(C507-Pad2)
- added copper zone on B.Cu, net Net-(C508-Pad1)
- added copper zone on F.Cu, net Net-(C508-Pad1)
- added copper zone on Power, net Net-(C508-Pad1)
- added copper zone on B.Cu, net Net-(C512-Pad1)
- added copper zone on F.Cu, net Net-(C512-Pad1)
- added copper zone on Power, net Net-(C513-Pad2)
- added copper zone on Power, net Net-(C515-Pad1)
- added copper zone on B.Cu, net Net-(C518-Pad1)
- added copper zone on F.Cu, net Net-(C518-Pad1)
- added copper zone on B.Cu, net Net-(D503-Pad1)
- added copper zone on F.Cu, net Net-(D503-Pad1)
- removed copper zone on Power, net GNDPWR
Other:
- board text added: "+24V"
- board text added: "+VOUT"
- board text added: "-VOUT"
- board text added: "ETH1CJTAG PROTOTYP V1.0 DEFAULT IP: 192.168.1.123 DEFAULT PORT: 2000 SHORT J1101 FOR DEFUALT MODE"
- board text added: "GND"
- board text added: "JT_GND"
- board text added: "JT_VCC"
- board text added: "RCTK"
- board text added: "SENSE"
- board text added: "SRST"
- board text added: "TCK"
- board text added: "TDI"
- board text added: "TDO"
- board text added: "TMS"
- board text added: "TRST"
- board text added: "nRESET"
- board text removed: "ETH1CJTAG PROTOTYP V1.0 IP: 192.168.1.123 PORT: 2000"
